File: Ergogen/output/pcbs/badWingsRight.kicad_pcb (KiCad board)
At the start: 2 copper layers, 147.6 x 109.7 mm, 154 parts

Commit message: Fix right half diode direction
Parts:
- turned D1 to -113 degrees
- turned D10 to -90 degrees
- turned D11 to -90 degrees
- turned D12 to -90 degrees
- turned D13 to -90 degrees
- turned D14 to -90 degrees
- turned D15 to -90 degrees
- turned D16 to -75 degrees
- turned D17 to -73 degrees
- turned D18 to -163 degrees
- turned D19 to -71 degrees
- turned D2 to -113 degrees
- turned D20 to -161 degrees
- turned D3 to -113 degrees
- turned D4 to -101 degrees
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